Commit message: feat: Navigation 仿真跑通 + 配置优化 + 文档完善
Navigation 仿真:
- nav2_params_sim 对齐 my_nav2_params，全向轮 min_y_velocity_threshold 0.001
- AMCL 粒子数 5000，recovery 启用，支持旋转 (max_vel_theta)
- costmap local 3×3m res 0.1，velocity_smoother 限速 0.5 m/s

仿真轻量化:
- Gazebo 物理 100Hz、关闭阴影
- Livox 点云 8000、update_rate 5Hz、downsample 2
- Fast-LIO point_filter_num 5、max_iteration 1、map_en false
- Ground segmentation n_bins 80、n_segments 180
- 新增 headless 模式 (headless:=True)

新增/修改:
- 仿真排障文档 rm_navigation_ws/docs/仿真启动排障.md
- pointcloud_to_laserscan_sim 脚本、bringup_sim headless 参数
- 无雷达测试脚本 run_test_a / run_test_a_headless / fake_sensors_for_test
- README 增加 5.9 Navigation 进度、5.10 下一步 TODO
- 决策树相关修改 (send_goal, is_detect_enemy 等)
- start_robot.sh、my_nav2_params.yaml

Co-authored-by: Cursor <cursoragent@cursor.com>

File: rm_navigation_ws/src/rm_simulation/livox_laser_simulation_RO2/urdf/mid360.xacro (robot description, xacro)
@@ -4,5 +4,6 @@
   <xacro:property name="laser_min_range" value="0.1"/>
   <xacro:property name="laser_max_range" value="200.0"/>
-  <xacro:property name="samples" value="30000"/>
+  <!-- 30000->8000 大幅降低点云密度，减轻 Fast-LIO/ground_seg 计算量 -->
+  <xacro:property name="samples" value="8000"/>
   <xacro:property name="resolution" value="0.002"/>
   <xacro:property name="noise_mean" value="0.0"/>
@@ -37,10 +38,10 @@
         <pose>0 0 0 0 0 0</pose>
         <visualize>true</visualize>
-        <update_rate>10</update_rate>
+        <update_rate>5</update_rate>
         <plugin name="${name}_plugin" filename="libros2_livox.so">
           <ray>
             <scan>
               <horizontal>
-                <samples>100</samples>
+                <samples>60</samples>
                 <resolution>1</resolution>
                 <min_angle>${0}</min_angle>
@@ -48,5 +49,5 @@
               </horizontal>
               <vertical>
-                <samples>360</samples>
+                <samples>180</samples>
                 <resolution>1</resolution>
                 <min_angle>${-7.22/180*M_PI}</min_angle>
@@ -67,5 +68,5 @@
           <visualize>false</visualize>
           <samples>${samples}</samples>
-          <downsample>1</downsample>
+          <downsample>2</downsample>
           <csv_file_name>$(find ros2_livox_simulation)/scan_mode/mid360.csv</csv_file_name>
           <topic>${topic}</topic>
